Commit message: Update grill_basket and grill_rack to revised STEP files
- grill_basket: DoubleGrillBasket2.step → DoubleGrillBasket.step (개정판,
  길이 542→532mm로 10mm 단축, 나머지 형상 동일)
- grill_rack: 구이 준비,완료 거치대.step → rag.step (치수 완전 동일한
  재추출본, 콜리전 보정값 그대로 유효)

Co-Authored-By: Claude Sonnet 5 <noreply@anthropic.com>

File: isaac_assets/urdf/grill_basket/grill_basket.urdf (robot description, URDF)
Before this commit: robot grill_basket, 1 links, 0 joints
Links:
- link base_link: geometry collision box size=0.532 0.339 0.0348; visual mesh filename=meshes/grill_basket.stl scale=1 1 1
