Commit message: Use upstream main a0509_stand

File: isaac_assets/urdf/a0509_stand/a0509_stand.urdf (robot description, URDF)
Before this commit: robot a0509_stand, 1 links, 0 joints
Links:
- link base_link: mass 40.0 -> 35.0; geometry collision box size=0.6 0.9 0.81; visual mesh filename=meshes/a0509_stand.stl scale=1 1 1
