Commit message: 로봇팔 제어기, 다이

File: isaac_assets/urdf/doosan_controller/doosan_controller.urdf (robot description, URDF)
Before this commit: robot doosan_controller, 1 links, 0 joints
Links:
- link base_link: geometry collision box size=0.482 0.228 0.342; visual mesh filename=meshes/doosan_controller.stl scale=1 1 1

Commit message: 컨트롤러

File: isaac_assets/urdf/doosan_controller/doosan_controller.urdf (robot description, URDF)
Before this commit: robot doosan_controller, 1 links, 0 joints
Links:
- link base_link: geometry collision box size=0.482 0.231 0.342; visual mesh filename=meshes/doosan_controller.stl scale=1 1 1
