Commit message: air_compressor_v2를 air_compressor로 통합
air_compressor.urdf 내부에 남아있던 v2 흔적(robot name, mesh 참조,
주석 헤더)을 실제 파일명에 맞게 정리하고, 중복된 air_compressor_v2
폴더를 삭제

File: isaac_assets/urdf/air_compressor/air_compressor.urdf (robot description, URDF)
Before this commit: robot air_compressor_v2, 1 links, 0 joints
Links:
- link base_link: geometry collision box size=0.4615 0.3126 0.5248; visual mesh filename=meshes/air_compressor.stl scale=1 1 1
